File: pcb/gamma_spectrometer/divider_board.kicad_sch (KiCad schematic)
At the start: 28 parts, among them Q401 MMBTA42, Q402 MMBTA42, Q403 MMBTA42, U402 ADA4817-1ARDZ

Commit message: pcb: делитель — R411 22 Ом на выходе TIA, +IN U402 на земле, обратная связь короче
- R411 = 22 Ом (RC0402FR-0722RL, 0402) между выводом 6 U402 и AMP_OUT, вплотную к
  выводу: R_SNUB против генерации TIA на ёмкостную нагрузку (кабель + вход шейпера).
- Вывод 3 U402 (+IN, опорная земля TIA) не был подключён — виа в паде на GND B.Cu.
- R417/C415 перенесены к выводам 1–2: петля обратной связи короче,
  паразитная C(анод↔FB) 0.13–0.22 → 0.05–0.09 пФ.
- Заливка перезалита; DRC по делителю: 0 нарушений зазора, схема↔плата 0.

Co-Authored-By: Claude Opus 5 (1M context) <noreply@anthropic.com>
Claude-Session: https://claude.ai/code/session_018uEKxzknn1WsQbGcTkkQF5
Parts:
- added R411: 22, Resistor_SMD:R_0402_1005Metric_Pad0.72x0.64mm_HandSolder, symbol Device:R
Connections:
- net AMP_OUT: now also R411.2; no longer U402.6 (OUT)
- new net: R411.1, U402.6 (OUT)
Changed lines of the file:
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@@
-	(wire
-		(pts
-			(xy 246.38 50.8) (xy 265.43 50.8)
-		)
-		(stroke
-			(width 0)
-			(type default)
-		)
-	)
 	(wire
 		(pts
@@
 		(pts
 			(xy 133.35 49.53) (xy 109.22 49.53)
+		)
+		(stroke
+			(width 0)
+			(type default)
+		)
+	)
+	(wire
+		(pts
+			(xy 246.38 50.8) (xy 257.81 50.8)
 		)
 		(stroke
@@
 					(unit 1)
 				)
+			)
+		)
+	)
+	(symbol
+		(lib_id "Device:R")
+		(at 261.62 50.8 90)
+		(unit 1)
+		(exclude_from_sim no)
+		(in_bom yes)
+		(on_board yes)
+		(dnp no)
+		(fields_autoplaced yes)
+		(property "Reference" "R411"
+			(at 261.62 44.45 90)
+			(effects
+				(font
+					(size 1.27 1.27)
+				)
+			)
+		)
+		(property "Value" "22"
+			(at 261.62 46.99 90)
+			(effects
+				(font
+					(size 1.27 1.27)
+				)
+			)
+		)
+		(property "Footprint" "Resistor_SMD:R_0402_1005Metric_Pad0.72x0.64mm_HandSolder"
+			(at 261.62 52.578 90)
+			(effects
+				(font
+					(size 1.27 1.27)
+				)
+				(hide yes)
+			)
+		)
+		(property "Datasheet" "~"
+			(at 261.62 50.8 0)
+			(effects
+				(font
+					(size 1.27 1.27)
+				)
+				(hide yes)
+			)
+		)
+		(property "Description" "Resistor"
+			(at 261.62 50.8 0)
+			(effects
+				(font
+					(size 1.27 1.27)
+				)
+				(hide yes)
+			)
+		)
+		(property "PN" "RC0402FR-0722RL"
+			(at 261.62 50.8 90)
+			(effects
+				(font
+					(size 1.27 1.27)
+				)
+				(hide yes)
+			)
+		)
+		(property "Ссылка на покупку " "https://www.electronshik.ru/item/YAG/RC0402FR-0722RL"
+			(at 261.62 50.8 90)
+			(effects
+				(font
+					(size 1.27 1.27)
+				)
+				(hide yes)
+			)
+		)
+		(pin "1"
+		)
+		(pin "2"
+		)
+		(instances
+			(project "gamma_spectrometer"
+				(path "/9de23c55-b97f-4e07-9aa5-29ce30f3c480/a23cd58c-c186-4cf3-8c49-bdaeee4d7f4c"
+					(reference "R411")
+					(unit 1)
+				)
