File: pcb/gamma_spectrometer/hv_board.kicad_sch (KiCad schematic)
At the start: 77 parts, among them Q201 IRLML0040, T201 ATB322524-0110-T000, U201 max1847eee+, U202 TL431DBZ

Commit message: Complete BOM: MPN and footprints for all components
Session 5 (2026-05-23) - full BOM assignment finished.

Components assigned (KiCad Symbol Fields + Footprints):
- 81 capacitors / 17 unique MPN (Yageo, Murata, Vishay, Holy Stone)
- 79 resistors / 28 unique MPN (Yageo RC/RT/RL/AC series)
- 3 inductors (Bourns SRN3015 + SRU5028)
- 2 LEDs (Foryard + Wurth 0805)
- 1 PTC fuse (MF-MSMF050-2)
- 1 ferrite bead (Murata BLM18EG121SN1D, 0603 - fixed from docs 0402)
- All active ICs (STM32G474, MAX1847, AD8000, FT231XQ, etc.)

Key design decisions:
- Standard bypass: 100nF X7R 0603 (easier hand soldering vs 0402)
- LED package 0805 (instead of 0402)
- C115 consolidated with C206 on single MPN (GRM32ER71A476KE15L)
- HV chain (1812 1kV X7R, 18x): Holy Stone C1812X104K102T
- AD8000 Cfb: GRM1555C1H1R0WA01D 1pF +/-0.05pF NP0
- R415: 50R -> 49.9R E96 (50R unavailable in catalog)
- L101/L102: SRN3015 (footprint Neosid SMS-ME3015, geometry verified)
- L103: SRU5028 (footprint L_Bourns_SRU5016, XY identical)

Documentation contradictions fixed:
- C115 MPN: GRM32ER61A476KE20L -> GRM32ER71A476KE15L
- FT231XS (SSOP-16) -> FT231XQ (QFN-20) - actual chip choice
- Tantalum MPN: TAJA106K016RNJ -> TR3B106K010C0750 (Vishay Low ESR)
- Inductor refs in usb_power_board_schematic.md updated

Remaining for PCB order:
- D202/D203 footprint: change SOD-123W -> SOD-123 (Diotec standard)
- J_PMT401: custom B14-38 footprint (during PCB layout)

Files:
- bom_fp_work.md - authoritative BOM with status, MPN, footprints, URLs
- pcb/gamma_spectrometer.net - fresh netlist with all MPN fields
- docs/session_context.md - session 5 final state

Co-Authored-By: Claude Sonnet 4.6 <noreply@anthropic.com>
Parts:
- C201: footprint (none) -> Capacitor_SMD:C_0805_2012Metric_Pad1.18x1.45mm_HandSolder; PN (none) -> CC0805JRX7R9BB333; Ссылка на покупку  (none) -> https://www.electronshik.ru/item/YAG/CC0805JRX7R9BB333
- C202: footprint (none) -> Capacitor_SMD:C_0805_2012Metric_Pad1.18x1.45mm_HandSolder; PN (none) -> CC0805JKX7R9BB474; Ссылка на покупку  (none) -> https://www.electronshik.ru/item/YAG/CC0805JKX7R9BB474
- C203, C207: footprint (none) -> Capacitor_SMD:C_0603_1608Metric_Pad1.08x0.95mm_HandSolder; PN (none) -> CC0603JRX7R9BB104; Ссылка на покупку  (none) -> https://www.electronshik.ru/item/YAG/CC0603JRX7R9BB104
- C204, C217: value 100nF -> 0.1uF; footprint (none) -> Capacitor_SMD:C_0603_1608Metric_Pad1.08x0.95mm_HandSolder; PN (none) -> CC0603JRX7R9BB104; Ссылка на покупку  (none) -> https://www.electronshik.ru/item/YAG/CC0603JRX7R9BB104
- C205: footprint (none) -> Capacitor_SMD:C_0603_1608Metric_Pad1.08x0.95mm_HandSolder; PN (none) -> CC0603JRNPO9BN101; Ссылка на покупку  (none) -> https://www.electronshik.ru/item/YAG/CC0603JRNPO9BN101
- C208: footprint (none) -> Capacitor_SMD:C_0603_1608Metric_Pad1.08x0.95mm_HandSolder; PN (none) -> CC0603KRX7R9BB103; Ссылка на покупку  (none) -> https://www.electronshik.ru/item/YAG/CC0603KRX7R9BB103
- D201: PN (none) -> BAS516
- D202, D203: footprint Diode_SMD:Nexperia_CFP3_SOD-123W -> Diode_SMD:D_SOD-123; PN (none) -> BZT52C18
- D204, D205, D206, D207, D208, D209, D210, D211: PN (none) -> BAV23S
- Q201: PN (none) -> IRLML0040; Ссылка на покупку  (none) -> https://www.electronshik.ru/item/HOTTECH/IRLML0040
- R201: footprint (none) -> Resistor_SMD:R_0603_1608Metric_Pad0.98x0.95mm_HandSolder; PN (none) -> RT0603BRD071ML; Ссылка на покупку  (none) -> https://www.electronshik.ru/item/YAG/RT0603BRD071ML
- R202: footprint (none) -> Resistor_SMD:R_0603_1608Metric_Pad0.98x0.95mm_HandSolder; PN (none) -> RC0603FR-07180KL; Ссылка на покупку  (none) -> https://www.electronshik.ru/item/YAG/RC0603FR-07180KL
- R203, R220, R231, R232: footprint (none) -> Resistor_SMD:R_0603_1608Metric_Pad0.98x0.95mm_HandSolder; PN (none) -> RC0603FR-07100KL; Ссылка на покупку  (none) -> https://www.electronshik.ru/item/YAG/RC0603FR-07100KL
- R204: footprint (none) -> Resistor_SMD:R_0603_1608Metric_Pad0.98x0.95mm_HandSolder; PN (none) -> RC0603FR-0710KL; Ссылка на покупку  (none) -> https://www.electronshik.ru/item/YAG/RC0603FR-0710KL
- R205: footprint (none) -> Resistor_SMD:R_0603_1608Metric_Pad0.98x0.95mm_HandSolder; PN (none) -> RL0603FR-070R1L; Ссылка на покупку  (none) -> https://www.electronshik.ru/item/YAG/RL0603FR-070R1L
- R206, R233: footprint (none) -> Resistor_SMD:R_0603_1608Metric_Pad0.98x0.95mm_HandSolder; PN (none) -> AC0603FR-0710RL; Ссылка на покупку  (none) -> https://www.electronshik.ru/item/YAG/AC0603FR-0710RL
- R207, R209, R210, R211, R212, R213, R214, R215, R216, R217: footprint (none) -> Resistor_SMD:R_1206_3216Metric_Pad1.30x1.75mm_HandSolder; PN (none) -> RC1206JR-07100ML; Ссылка на покупку  (none) -> https://www.electronshik.ru/item/YAG/RC1206JR-07100ML
- R208: footprint (none) -> Resistor_SMD:R_0603_1608Metric_Pad0.98x0.95mm_HandSolder; PN (none) -> RC0603FR-072M2L; Ссылка на покупку  (none) -> https://www.electronshik.ru/item/YAG/RC0603FR-072M2L
- R218: footprint (none) -> Resistor_SMD:R_0603_1608Metric_Pad0.98x0.95mm_HandSolder; PN (none) -> RC0603FR-071K2L; Ссылка на покупку  (none) -> https://www.electronshik.ru/item/YAG/RC0603FR-071K2L
- R219: footprint (none) -> Resistor_SMD:R_0603_1608Metric_Pad0.98x0.95mm_HandSolder; PN (none) -> RC0603FR-07110KL; Ссылка на покупку  (none) -> https://www.electronshik.ru/item/YAG/RC0603FR-07110KL
- R221, R222, R223, R224, R225, R226, R227, R228, R229, R230: footprint (none) -> Resistor_SMD:R_1206_3216Metric_Pad1.30x1.75mm_HandSolder; PN (none) -> RC1206FR-076M8L; Ссылка на покупку  (none) -> https://www.electronshik.ru/item/YAG/RC1206FR-076M8L
- T201: PN (none) -> ATB322524-0110-T000
- U201: PN (none) -> max1847eee+
- U202: value TL431DBZ -> TL431; PN (none) -> TL431; Ссылка на покупку  (none) -> https://www.electronshik.ru/item/YOUTAI/TL431

Commit message: pcb: Q201 IRLML0040 → IRLML0060 (60 В) — запас по выбросу стока
Ключ обратноходового преобразователя ВВ-платы: та же посадка SOT-23 и
распиновка (1-G, 2-S, 3-D). Пик на стоке по расчёту 38.8 В типично,
43–45 В в худшем случае — у IRLML0040 (40 В, лавина не нормирована)
запаса не было. Снаббер BAS516 + C208 + 2×BZT52C18 без изменений.
Схема↔плата: 0 расхождений.

Co-Authored-By: Claude Opus 5 (1M context) <noreply@anthropic.com>
Claude-Session: https://claude.ai/code/session_018uEKxzknn1WsQbGcTkkQF5
Parts:
- Q201: value IRLML0040 -> IRLML0060; PN IRLML0040 -> IRLML0060; Ссылка на покупку  https://www.electronshik.ru/item/HOTTECH/IRLML0040 -> https://www.electronshik.ru/item/HOTTECH/IRLML0060
Changed lines of the file:
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@@
 			)
 		)
-		(property "Value" "IRLML0040"
+		(property "Value" "IRLML0060"
 			(at 156.21 114.2999 0)
 			(effects
@@
 			)
 		)
-		(property "PN" "IRLML0040"
+		(property "PN" "IRLML0060"
 			(at 149.86 113.03 0)
 			(effects
@@
 			)
 		)
-		(property "Ссылка на покупку " "https://www.electronshik.ru/item/HOTTECH/IRLML0040"
+		(property "Ссылка на покупку " "https://www.electronshik.ru/item/HOTTECH/IRLML0060"
 			(at 149.86 113.03 0)
 			(effects

Commit message: hv: C_COMP2 на плате, перенумерация конденсаторов, проверка земли платы ВВ
Плата и схема (правки пользователя):
- C201 = 22 пФ C0G (C_COMP2) с вывода COMP MAX1847 на GND — по итогам расчёта наводки;
- перенумерация конденсаторов платы ВВ: прежние C201…C217 → C202…C218;
- восстановлена дорожка R201→C202 (без неё запас по фазе падал с 80° до 32°);
- подключён вывод 16 U201 (SYNC) — висел в воздухе;
- сшита земля платы: выводы 10/11/12 MAX1847, R205 и C207 были отделены от вторички,
  умножителя и цепи коррекции, соединялись только через межплатные цанги;
- подключён земляной вывод C211 (возврат умножителя).
Итог по DRC: нарушений зазоров 23 → 4, разрывов земли на плате ВВ — 0.

Документация:
- обновлены все обозначения под новую нумерацию (доки, BOM, шпаргалка, скрипты расчёта);
- C209 (снаббер, 10 нФ) в BOM на 50 В, а узел под ним на 35.7 В с пиками 38–45 В: нужен 100 В;
- C210–C217 (1 нФ 500 В): размах на ступень 310…385 В, запас 1.3× при уставке 1500 В
  (прежняя оценка «189 В» шла из ошибочных 8 ступеней);
- корпуса в BOM платы ВВ приведены к реальным (0603/0805 вместо 0402);
- .net перевыгружен: 178 компонентов.

Осталось: дорожка Net-(C18a201-Pad2) не доходит 0.588 мм до пада C18a201.2 (ВЧ-фильтр
выхода разомкнут), 4 ВВ-зазора, терморазгрузка C202, шелкография.

Co-Authored-By: Claude Opus 5 (1M context) <noreply@anthropic.com>
Claude-Session: https://claude.ai/code/session_018uEKxzknn1WsQbGcTkkQF5
Parts:
- added C201: 22pF, Capacitor_SMD:C_0402_1005Metric_Pad0.74x0.62mm_HandSolder, symbol Device:C
- renumbered C201 to C202, C202 to C203, C203 to C204, C204 to C205, C205 to C206, C206 to C207, C207 to C208, C208 to C209, C209 to C210, C210 to C211, C211 to C212, C212 to C213, C213 to C214, C214 to C215, C215 to C216, C216 to C217, C217 to C218
Connections:
- net GND: now also C201.1
- net at R201.1, U201.4 (COMP): now also C201.2
Other:
- moved on the sheet: C202, R201
