File: pcb/gamma_spectrometer/gamma_spectrometer.kicad_pcb (KiCad board)
At the start: 2 copper layers, 255 x 45 mm, 232 parts, among them J101 DX07S024WJ3R400, Q201 IRLML0060, Q401 MMBTA42, Q402 MMBTA42, Q403 MMBTA42, T201 ATB322524-0110-T000, U101 LP5907MFX-3.3, U102 AMS1117-3.3, U103 FT231XQ, U104 TPS60400DBV, U201 max1847eee+, U202 TL431, U301 REF35250QDBVR, U302 STM32G474MET6, U303 W25Q64JVSSIQ, U402 ADA4817-1ARDZ, Y301 ABM8G-16.000MHZ-4Y-T3

Commit message: pcb: четыре платы собраны в одну заготовку с перемычками под разлом
pcb/panelize.py: шаг плат 70 -> 47.5 мм (зазор 2.5 мм под стандартную фрезу),
заготовка 187.5 x 45 мм вместо 265 x 55. Перенос только по X, без поворотов.

Контур: 4 окружности заменены на 12 дуг и 12 прямых сторон перемычек.
Перемычки — 6 штук, по две на стык под ±15° от линии центров, ширина 3 мм,
длина 4.0 мм. Отверстия разлома — 36 шт Ø0.6 NPTH, по 3 в ряд с шагом 1 мм,
центры вынесены на 0.2 мм наружу контура, чтобы до меди осталось 0.402 мм при
норме выреза вокруг NPTH 0.3.

Шесть зон запрета заливки по перемычкам: контуры зон GND нарисованы крупнее
платы (их обрезал круглый Edge.Cuts), без запрета перезаливка залила бы медь
в перемычки и на отверстия разлома.

Заодно: сверло стоек 2.75 -> 2.8 мм, проход -ВВ H_HV301 Ø5.0 -> Ø4.5 (не нужна
фрезеровка, вырез в полигоне стал 0.50 мм, провод Ø3 проходит с зазором 0.75 мм
по радиусу). Футпринт переименован в HOLE_HV_WIRE_D4.5, библиотека обновлена.
Вся сверловка теперь в номинальном ряду завода, 8 типов.

Проверено: геометрия каждой платы относительно своего центра совпадает с
исходной до нуля (33986 точек суммарно); DRC даёт те же 3 зазора и 27
«не соединено»; медь до контура 0.501 мм; радиусы дуг 22.500.

Перед выпуском в KiCad: перезалить зоны (снимет 6 items_not_allowed от старой
заливки на зонах запрета), поменять класс Default на 0.8/0.3, перевыгрузить
герберы.

Co-Authored-By: Claude Opus 5 (1M context) <noreply@anthropic.com>
Claude-Session: https://claude.ai/code/session_018uEKxzknn1WsQbGcTkkQF5
Parts:
- added PANEL1: PANEL_MOUSEBITES, PANEL_MOUSEBITES, F.Cu at (0.00, 0.00)
- moved COAX4 67.5 mm to (240.8, 100.5)
- moved REF** 67.5 mm to (229.1, 85.1)
- moved REF** 67.5 mm to (235.7, 118.8)
- moved REF** 67.5 mm to (226.1, 88.5)
- moved C408 67.5 mm to (238.0, 90.5)
- moved C409 67.5 mm to (243.5, 90.5)
- moved C410 67.5 mm to (249.0, 91.5)
- moved C411 67.5 mm to (248.5, 102.8)
- moved C412 67.5 mm to (250.2, 103.0)
- moved C413 67.5 mm to (243.5, 104.0)
- moved C414 67.5 mm to (243.5, 102.5)
- moved C415 67.5 mm to (254.0, 103.2)
- moved COAX2 67.5 mm to (242.8, 99.2)
- moved D401 67.5 mm to (238.0, 94.0)
- moved D402 67.5 mm to (241.5, 90.5)
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Routing:
- net /USB_Power_Board/D_N: track 12.9 -> 14.3 mm
- net LED: track 56.1 -> 57.5 mm
- net +3.3V_D: track 161.1 -> 162.4 mm
- net Net-(U302-PA5): track 20.1 -> 21.3 mm
- net GND: track 23.1 -> 24.1 mm
- net Net-(U302-PA1): track 13.5 -> 14.0 mm
- net Net-(C210-Pad1): track 2.17 -> 1.67 mm
- net (no net): vias 1 -> 0
Other:
- board size 255 x 45 mm -> 187.5 x 45 mm
