File: pcb/gamma_spectrometer/gamma_spectrometer.kicad_pcb (KiCad board)
At the start: 2 copper layers, 187.5 x 45 mm, 233 parts, among them J101 DX07S024WJ3R400, Q201 IRLML0060, Q401 MMBTA42, Q402 MMBTA42, Q403 MMBTA42, T201 ATB322524-0110-T000, U101 LP5907MFX-3.3, U102 AMS1117-3.3, U103 FT231XQ, U104 TPS60400DBV, U201 max1847eee+, U202 TL431, U301 REF35250QDBVR, U302 STM32G474MET6, U303 W25Q64JVSSIQ, U402 ADA4817-1ARDZ, Y301 ABM8G-16.000MHZ-4Y-T3

Commit message: pcb: плата МК на LQFP-48 (STM32G474CBT6), герберы перевыгружены
Схема и плата МК переразведены под STM32G474CBT6 в LQFP-48 7x7 вместо
STM32G474MET6 в LQFP-80 12x12. Заказ MCT6TR отменён поставщиком из-за
пересорта; CBT6 есть в наличии за 238 руб против 1410 и 6 недель.
Все 24 задействованных вывода есть и в LQFP-48.

Снесены 289 дорожек и 127 виа в круге (195, 100) R22.5, разведено заново.
Удалены C304 и C309 — лишние пары развязки (выводов питания стало 4 из 6).
Падам VSSA/VSS 19/23/35/47 выставлено zone_connect = 2: при шаге 0.5 мм
два мостика терморазгрузки не влезают, сплошное соединение заодно даёт
минимальную индуктивность возврата.

Контур заготовки не менялся: Edge_Cuts байт в байт как в версии, по которой
выставлен счёт N 19696. Сверловка плат USB, ВВ и делителя идентична прежней.
Компонентов 178 -> 176, цепей 118 без изменений, ERC 0 ошибок.

Попутно закрыто:
- 5 виа с пояском 0.15 мм. Корень не в разводке, а в настройке проекта:
  класс Default держал via_diameter = 0.6, а min_via_annular_width = 0.1,
  поэтому каждая новая виа выходила бракованной молча. Теперь 0.8 и 0.25.
- Плата МК потеряла посадочное место стоек STANDOFF_M2.5_GND_x3_TRIANGLE
  (три отверстия D2.8 крепления стека) — оно стоит ровно в центре и ушло
  вместе с выделением при сносе разводки. Нашлось сравнением сверловки
  по платам: D2.80 было 12, стало 9. Восстановлено из HEAD байт в байт.
- Замыкание GND на UART_TX — следствие предыдущего: пока стоек не было,
  дорожка на B.Cu легла через их пад на 330 градусах.
- Оторванный остров заливки под R311: нижнее плечо делителя PGA x4 было
  фактически не заземлено.
- Разрыв дорожки у C18a201 на плате ВВ (ВЧ-фильтр выхода был разомкнут).
- Дублирующая дорожка +3.3V_D на плате USB.

DRC: 413 нарушений, по делу 3 принятых ВВ-правила. Замыканий, мостиков
маски, висячих дорожек и неполных терморазгрузок 0. Не соединено 26 =
25 межплатных (мост — цанг-пины в стеке) + одна старая пара зон на USB.
Виа 210, поясок 0.250 у всех. Сверловка сверена с пла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
Parts:
- removed C304, C309: 0.1uF, Capacitor_SMD:C_0603_1608Metric_Pad1.08x0.95mm_HandSolder
- U302: value STM32G474MET6 -> STM32G474CBT6; footprint Package_QFP:LQFP-80_12x12mm_P0.5mm -> Package_QFP:LQFP-48_7x7mm_P0.5mm
- moved C306 17.4 mm to (200.5, 93.0), turned to 0 degrees
- moved C305 6.54 mm to (189.2, 103.0), turned to 180 degrees
- moved C307 4.51 mm to (199.8, 106.5)
- moved C318 3.40 mm to (190.5, 89.8), turned to -90 degrees
- moved R307 3.26 mm to (192.2, 92.2), turned to 0 degrees
- moved C312 3.06 mm to (197.5, 107.8)
- moved R302 3.06 mm to (196.0, 107.8)
- moved R311 3.01 mm to (188.5, 97.5), turned to 180 degrees
- moved U302 1.46 mm to (196.2, 99.2)
- moved C308 0.90 mm to (202.8, 95.2), turned to 90 degrees
- moved C317 0.44 mm to (196.0, 91.0)
- moved R308 0.39 mm to (197.2, 88.5)
Connections:
- U302 pad 10: unconnected-(U302-PC2-Pad10) -> Net-(U302-PA2)
- U302 pad 11: unconnected-(U302-PC3-Pad11) -> Net-(U302-PA3)
- U302 pad 12: HV_MONITOR -> DAC_TEST
- U302 pad 13: Net-(U302-PA1) -> Net-(U302-PA5)
- U302 pad 14: Net-(U302-PA2) -> Net-(U302-PA6)
- U302 pad 15: GND -> Net-(U302-PA1)
- U302 pad 16: +3.3V_D -> Net-(U302-PB0)
- U302 pad 17: Net-(U302-PA3) -> unconnected-(U302-PB1-Pad17)
- U302 pad 18: DAC_TEST -> unconnected-(U302-PB2-Pad18)
- U302 pad 19: Net-(U302-PA5) -> GND
- U302 pad 20: Net-(U302-PA6) -> Net-(U301-VREF)
- U302 pad 21: Net-(U302-PA1) -> Net-(U302-VDDA)
- U302 pad 22: unconnected-(U302-PC4-Pad22) -> HV_ENABLE
- U302 pad 23: unconnected-(U302-PC5-Pad23) -> GND
- U302 pad 24: Net-(U302-PB0) -> +3.3V_D
- U302 pad 26: unconnected-(U302-PB2-Pad26) -> TSENS_IN
- U302 pad 27: GND -> unconnected-(U302-PB13-Pad27)
- U302 pad 28: Net-(U301-VREF) -> unconnected-(U302-PB14-Pad28)
- U302 pad 29: Net-(U302-VDDA) -> unconnected-(U302-PB15-Pad29)
- U302 pad 30: unconnected-(U302-PE7-Pad30) -> Net-(U302-PA8)
- U302 pad 31: unconnected-(U302-PE8-Pad31) -> UART_RX
- U302 pad 32: unconnected-(U302-PE9-Pad32) -> UART_TX
- U302 pad 35: unconnected-(U302-PE12-Pad35) -> GND
- U302 pad 36: unconnected-(U302-PE13-Pad36) -> +3.3V_D
- U302 pad 37: unconnected-(U302-PE14-Pad37) -> SWDIO
- U302 pad 38: unconnected-(U302-PE15-Pad38) -> SWCLK
- U302 pad 39: HV_ENABLE -> SPI_CS
- U302 pad 40: GND -> SPI_SCK
- U302 pad 41: +3.3V_D -> SPI_MISO
- U302 pad 42: unconnected-(U302-PB11-Pad42) -> SPI_MOSI
- U302 pad 43: TSENS_IN -> LED
- U302 pad 47: unconnected-(U302-PD8-Pad47) -> GND
- U302 pad 48: unconnected-(U302-PD9-Pad48) -> +3.3V_D
- U302 pad 8: unconnected-(U302-PC0-Pad8) -> HV_MONITOR
- U302 pad 9: unconnected-(U302-PC1-Pad9) -> Net-(U302-PA1)
Routing:
- net +3.3V_D: track 162.4 -> 139.3 mm, vias 6 -> 5
- net Net-(C312-Pad1): track 32.5 -> 27.0 mm
- net Net-(U302-PA6): track 6.53 -> 11.5 mm
- net Net-(U302-PB0): track 9.07 -> 13.6 mm
- net TSENS_IN: track 13.4 -> 17.6 mm
- net Net-(U301-VREF): track 26.6 -> 29.8 mm
- net HV_MONITOR: track 46.0 -> 42.9 mm, vias 0 -> 2
- net HV_ENABLE: track 19.8 -> 22.5 mm, vias 2 -> 1
- net GND: track 24.1 -> 21.4 mm, vias 170 -> 157
- net Net-(U302-VDDA): track 10.9 -> 13.3 mm
- net Net-(U302-PA3): track 8.28 -> 10.5 mm
- net SPI_MISO: track 10.6 -> 12.7 mm
- net Net-(U302-PF0): track 7.60 -> 9.69 mm
- net Net-(U302-PF1): track 6.71 -> 8.80 mm
- net Net-(U302-PA1): track 14.0 -> 15.8 mm
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